File: Valpo-PCB-Ruler.kicad_pcb (KiCad board)
At the start: 2 copper layers, 203.2 x 38.1 mm, 52 parts

Commit message: Update constants
Other:
- board text added: "Boltzmann Const.(k )= 1.381×10 J/K"
- board text added: "Vacuum Permittivity(ε )=8.854×10 F/m"
- board text removed: "-1"
- board text removed: "Boltzmann Const.(k )= 1.381×10 JK"
- board text removed: "Electron Volt(eV)=1.602×10 J"
- board text removed: "Vacuum Permittivity(ε )=8.854×10 Fm"
Changed lines of the file:
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@@
   (general
     (thickness 1.6)
-    (drawings 1236)
+    (drawings 1232)
     (tracks 20)
     (zones 0)
@@
   (layers
     (0 F.Cu signal hide)
-    (31 B.Cu signal hide)
+    (31 B.Cu signal)
     (32 B.Adhes user hide)
     (33 F.Adhes user hide)
@@
     (36 B.SilkS user)
     (37 F.SilkS user hide)
-    (38 B.Mask user)
+    (38 B.Mask user hide)
     (39 F.Mask user hide)
     (40 Dwgs.User user)
@@
       (xy -4.88682 -4.482967) (xy -4.876452 -4.486047) (xy -4.871357 -4.484994)) (layer F.SilkS) (width 0.01))
   )
-  (gr_text -31 (at 125.73 78.2955) (layer B.SilkS)
+  (gr_text -31 (at 125.73 65.5955) (layer B.SilkS)
     (effects (font (size 0.75 0.75) (thickness 0.15)) (justify mirror))
   )
-  (gr_text "Mass of an Electron=9.109×10  kg" (at 150.122429 79.20847) (layer B.SilkS)
+  (gr_text "Mass of an Electron=9.109×10  kg" (at 149.86 66.675) (layer B.SilkS)
     (effects (font (size 1 1) (thickness 0.15)) (justify left mirror))
   )
-  (gr_text "Speed of Sound=343m/s" (at 150.122429 84.2073) (layer B.SilkS)
+  (gr_text "Speed of Sound=343m/s" (at 149.86 81.915) (layer B.SilkS)
     (effects (font (size 1 1) (thickness 0.15)) (justify left mirror))
   )
@@
   (gr_line (start 228.464 79.2965) (end 218.2495 79.2965) (layer B.SilkS) (width 0.12))
   (gr_line (start 250.435 80.9475) (end 245.609 80.9475) (layer B.SilkS) (width 0.12))
-  (gr_text -6 (at 122.555 75.692) (layer B.SilkS)
+  (gr_text -6 (at 121.92 75.692) (layer B.SilkS)
     (effects (font (size 0.75 0.75) (thickness 0.15)) (justify mirror))
   )
@@
     (effects (font (size 0.75 0.75) (thickness 0.15)) (justify mirror))
   )
-  (gr_text "Vacuum Permeability(μ )=1.257×10 H/m" (at 134.142667 76.709056) (layer B.SilkS)
-    (effects (font (size 1 1) (thickness 0.15)) (justify mirror))
-  )
-  (gr_text -1 (at 119.9515 73.279) (layer B.SilkS)
-    (effects (font (size 0.75 0.75) (thickness 0.15)) (justify mirror))
-  )
-  (gr_text -12 (at 123.19 73.279) (layer B.SilkS)
-    (effects (font (size 0.75 0.75) (thickness 0.15)) (justify mirror))
-  )
-  (gr_text "Vacuum Permittivity(ε )=8.854×10  Fm" (at 134.904572 74.209642) (layer B.SilkS)
-    (effects (font (size 1 1) (thickness 0.15)) (justify mirror))
+  (gr_text "Vacuum Permeability(μ )=1.257×10 H/m" (at 149.86 76.835) (layer B.SilkS)
+    (effects (font (size 1 1) (thickness 0.15)) (justify left mirror))
   )
-  (gr_text -19 (at 128.143 68.2475) (layer B.SilkS)
+  (gr_text -12 (at 122.555 73.279) (layer B.SilkS)
     (effects (font (size 0.75 0.75) (thickness 0.15)) (justify mirror))
   )
-  (gr_text "Electron Volt(eV)=1.602×10  J" (at 150.122429 69.210814) (layer B.SilkS)
+  (gr_text "Vacuum Permittivity(ε )=8.854×10   F/m" (at 149.86 74.295) (layer B.SilkS)
     (effects (font (size 1 1) (thickness 0.15)) (justify left mirror))
   )
-  (gr_text "Speed of Light(c)=2.998×10 m/s" (at 150.122429 81.707884) (layer B.SilkS)
+  (gr_text "Speed of Light(c)=2.998×10 m/s" (at 149.86 79.375) (layer B.SilkS)
     (effects (font (size 1 1) (thickness 0.15)) (justify left mirror))
   )
-  (gr_text 8 (at 127.6985 80.8355) (layer B.SilkS)
+  (gr_text 8 (at 127.635 78.74) (layer B.SilkS)
     (effects (font (size 0.75 0.75) (thickness 0.15)) (justify mirror))
   )
@@
     (effects (font (size 0.75 0.75) (thickness 0.15)) (justify mirror))
   )
-  (gr_text -1 (at 121.031 70.739) (layer B.SilkS)
-    (effects (font (size 0.75 0.75) (thickness 0.15)) (justify mirror))
-  )
-  (gr_text "Boltzmann Const.(k )= 1.381×10  JK" (at 150.122429 71.710228) (layer B.SilkS)
+  (gr_text "Boltzmann Const.(k )= 1.381×10  J/K" (at 149.86 71.755) (layer B.SilkS)
     (effects (font (size 1 1) (thickness 0.15)) (justify left mirror))
   )
-  (gr_text -23 (at 124.0155 70.739) (layer B.SilkS)
+  (gr_text -23 (at 123.825 70.739) (layer B.SilkS)
     (effects (font (size 0.75 0.75) (thickness 0.15)) (justify mirror))
   )
-  (gr_text -19 (at 124.6505 65.7075) (layer B.SilkS)
+  (gr_text -19 (at 124.6505 68.2475) (layer B.SilkS)
     (effects (font (size 0.75 0.75) (thickness 0.15)) (justify mirror))
   )
-  (gr_text "Elementary Charge(q)=1.602×10  C" (at 150.122429 66.7114) (layer B.SilkS)
+  (gr_text "Elementary Charge(q)=1.602×10  C" (at 149.86 69.215) (layer B.SilkS)
     (effects (font (size 1 1) (thickness 0.15)) (justify left mirror))
   )
