File: Valpo-PCB-Ruler.kicad_pcb (KiCad board)
At the start: 2 copper layers, 203.2 x 38.1 mm, 52 parts

Commit message: Move BGA, add blank copper for name
Parts:
- removed BGA 20x20 1.0mm Pitch: BGA-400_21.0x21.0mm_Layout20x20_P1.0mm, Package_BGA:BGA-400_21.0x21.0mm_Layout20x20_P1.0mm
- added BGA 0.8mm: BGA-48_8.0x9.0mm_Layout6x8_P0.8mm, Package_BGA:BGA-48_8.0x9.0mm_Layout6x8_P0.8mm, B.Cu at (206.8, 83.3)
Other:
- board text added: "fabid: JLCJLCJLCJLC"
